File: board/_autosave-lora2040.kicad_sch (KiCad schematic)
At the start: 46 parts, among them J1 u.FL, J2 USB_B_Micro, J3 Conn_01x04, U1 SX1262IMLTRT, U2 BGS12WN6E6327, U3 0900FM15K0039, U4 MR20H40 or AS3004204, U5 RP2040, U6 RTX-2016BD32-S-32.000-TR, Y2 ABM8-272-T3

Commit message: seeing what castelations look like
Parts:
- added C24, C26: 1uF, Capacitor_SMD:C_0402_1005Metric, symbol Device:C
- added C25: 10nF, Capacitor_SMD:C_0402_1005Metric, symbol Device:C
- added U7: TPS73633DBV, Package_TO_SOT_SMD:SOT-23-5, symbol Regulator_Linear:TPS73633DBV
Connections:
- net VDD_RF is gone; now on net +3V3: C16.1, C18.1, U1.1 (VDD_IN), U1.10 (VBAT), U1.11 (VBAT_IO)
- net +3V3: now also C24.2, U7.5 (OUT)
- net GND: now also C24.1, C25.1, C26.1, U7.2 (GND)
- net VUSB: now also C26.2, U7.1 (IN), U7.3 (EN)
- new net: C25.2, U7.4 (NR)
Other:
- note added: "VDD_RF"
- moved on the sheet: C1, C10, C11, C12, C13, C14, C15, C16, C17, C18, C19, C2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
