File: board/lora2040.kicad_sch (KiCad schematic)
At the start: 46 parts, among them J1 u.FL, J2 USB_B_Micro, J3 Conn_01x04, U1 SX1262IMLTRT, U2 BGS12WN6E6327, U3 0900FM15K0039, U4 MR20H40 or AS3004204, U5 RP2040, U6 RTX-2016BD32-S-32.000-TR, Y2 ABM8-272-T3

Commit message: routing tests
Parts:
- added C24, C26: 1uF, Capacitor_SMD:C_0402_1005Metric, symbol Device:C
- added C25: 10nF, Capacitor_SMD:C_0402_1005Metric, symbol Device:C
- added C27: 10uF, Capacitor_SMD:C_0402_1005Metric, symbol Device:C
- added U7: TPS73633DBV, Package_TO_SOT_SMD:SOT-23-5, symbol Regulator_Linear:TPS73633DBV
- R2, R5: footprint custom-footprints:sx126x_R_0201 -> Resistor_SMD:R_0402_1005Metric
Connections:
- net VDD_RF is gone; now on net +3V3: C16.1, C18.1, U1.1 (VDD_IN), U1.10 (VBAT), U1.11 (VBAT_IO)
- net +3V3: now also C24.2, C27.2, U7.5 (OUT)
- net GND: now also C24.1, C25.1, C26.1, C27.1, U7.2 (GND)
- net VUSB: now also C26.2, U7.1 (IN), U7.3 (EN)
- net UART0_TX: now reaches U5.2 (GPIO0)
- net UART0_RX: now reaches U5.3 (GPIO1)
- net I2C0_SDA: now reaches U5.6 (GPIO4)
- net I2C0_SCL: now reaches U5.7 (GPIO5)
- net ANT_SW renamed RF_SW_PWR
- new net: C25.2, U7.4 (NR)
Other:
- note added: "NOTE: ENOB=8 =0.41V?"
- note added: "VDD_RF"
- note removed: "NOTE: ENOB=8"
- moved on the sheet: C1, C10, C11, C12, C13, C14, C15, C16, C17, C18, C19, C2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

Commit message: BOM clean up and routing
Parts:
- added D1: LED, LED_SMD:LED_0402_1005Metric, symbol Device:LED
- added J4: Conn_01x01, custom-footprints:castellated_07mm, symbol Connector_Generic:Conn_01x01
- added J5: Conn_01x02, Connector_PinHeader_1.00mm:PinHeader_1x02_P1.00mm_Vertical, symbol Connector_Generic:Conn_01x02
- added J6: Conn_02x06_Odd_Even, Connector_PinHeader_1.00mm:PinHeader_2x06_P1.00mm_Vertical, symbol Connector_Generic:Conn_02x06_Odd_Even
- added J8: Conn_01x04, Connector_PinHeader_1.00mm:PinHeader_1x04_P1.00mm_Vertical, symbol Connector_Generic:Conn_01x04
- added R11: 1K, custom-footprints:sx126x_R_0201, symbol Device:R_US
- FB1: Manufacturer (none) -> Murata Electronics; Part Number (none) -> BLM15PG100SN1D
- J3: now not fitted; now left out of the parts list
- L1: value 47nF -> 47nH; Manufacturer (none) -> Murata Electronics; Part Number (none) -> LQW15AN47NJ00D
- L7: Manufacturer (none) -> TDK Corporation; Part Number (none) -> MLZ2012M150WT000
- U1: Manufacturer (none) -> Semtech Corporation; Part Number (none) -> SX1262IMLTRT
- U2: Manufacturer (none) -> Infineon Technologies; Part Number (none) -> BGS12WN6E6327
- U3: value 0900FM15K0039 -> 0900FM15K0039001E; Manufacturer (none) -> Johanson Technology Inc.; Part Number (none) -> 0900FM15K0039001E
- U4: Manufacturer (none) -> Avalanche Technology; Part Number (none) -> AS3004204-0054X0PWAY
- U5: Manufacturer (none) -> Raspberry Pi; Part Number (none) -> SC0914
- U6: Manufacturer (none) -> Raltron Electronics; Part Number (none) -> RTX-2016BD32-S-32.000-TR
- U7: value TPS73633DBV -> TPS73633DBV or MIC5219-3.3YM5-TR?; Manufacturer (none) -> Microchip Technology; Part Number (none) -> MIC5219-3.3YM5-TR
- Y2: Manufacturer (none) -> Abracon LLC; Part Number (none) -> ABM8-272-T3
Connections:
- net +3V3: now also J6.7 (Pin_7), J8.4 (Pin_4)
- net GND: now also D1.1 (K), J5.1 (Pin_1), J6.5 (Pin_5), J6.6 (Pin_6), J8.1 (Pin_1)
- net I2C0_SCL: now also J6.4 (Pin_4)
- net I2C0_SDA: now also J6.2 (Pin_2)
- net UART0_RX: now also J6.1 (Pin_1)
- net UART0_TX: now also J6.3 (Pin_3)
- net SWCLK: now reaches U5.24 (SWCLK)
- net SWCLK: now also J8.2 (Pin_2)
- net SWD: now reaches U5.25 (SWD)
- net SWD: now also J8.3 (Pin_3)
- net LED: now reaches U5.35 (GPIO23)
- net LED: now also R11.1
- net ADC0: now reaches U5.38 (GPIO26_ADC0)
- net ADC0: now also J6.12 (Pin_12)
- net ADC1: now reaches U5.39 (GPIO27_ADC1)
- net ADC1: now also J6.10 (Pin_10)
- net ADC2: now reaches U5.40 (GPIO28_ADC2)
- net ADC2: now also J6.8 (Pin_8)
- net VUSB renamed VBUS
- net VBUS: now also J4.1 (Pin_1), J5.2 (Pin_2)
- new net: D1.2 (A), R11.2
Other:
- moved on the sheet: C5, C6, C7

Commit message: schematic cleanup and BOM
Parts:
- C24: value 1uF -> 10uF
- C25: value 10nF -> 470pF
Other:
- note added: "Eventually use castellations"
- note added: "Temporary breakout header"
- moved on the sheet: J4, J5, J6
Changed lines of the file:
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@@
 		)
 	)
+	(rectangle
+		(start 188.595 43.18)
+		(end 285.115 73.66)
+		(stroke
+			(width 0)
+			(type default)
+		)
+		(fill
+			(type none)
+		)
+	)
 	(text "0.8mm pitch JST SUR series\n32AWG"
 		(exclude_from_sim no)
@@
 		)
 	)
+	(text "Temporary breakout header"
+		(exclude_from_sim no)
+		(at 212.344 46.482 0)
+		(effects
+			(font
+				(size 1.905 1.905)
+			)
+		)
+	)
 	(text "Close to\npin 45"
 		(exclude_from_sim no)
@@
 		)
 	)
+	(text "Eventually use castellations"
+		(exclude_from_sim no)
+		(at 263.398 46.736 0)
+		(effects
+			(font
+				(size 1.905 1.905)
+			)
+		)
+	)
 	(text "short for\nbootloader"
 		(exclude_from_sim no)
@@
 	)
 	(label "UART0_RX"
-		(at 87.63 171.45 180)
+		(at 200.66 54.61 180)
 		(fields_autoplaced yes)
 		(effects
@@
 	)
 	(label "RF_DIO3"
-		(at 172.72 134.62 180)
+		(at 173.99 134.62 180)
 		(fields_autoplaced yes)
 		(effects
@@
 	)
 	(label "ADC0"
-		(at 100.33 184.15 0)
+		(at 213.36 67.31 0)
 		(fields_autoplaced yes)
 		(effects
@@
 	)
 	(label "VBUS"
-		(at 35.56 177.8 0)
+		(at 266.7 55.88 0)
 		(fields_autoplaced yes)
 		(effects
@@
 	)
 	(label "UART0_TX"
-		(at 87.63 173.99 180)
+		(at 200.66 57.15 180)
 		(fields_autoplaced yes)
 		(effects
@@
 	)
 	(label "ADC2"
-		(at 100.33 179.07 0)
+		(at 213.36 62.23 0)
 		(fields_autoplaced yes)
 		(effects
@@
 	)
 	(label "VBUS"
-		(at 55.88 173.99 180)
+		(at 227.33 53.34 180)
 		(fields_autoplaced yes)
 		(effects
@@
 	)
 	(label "ADC1"
-		(at 100.33 181.61 0)
+		(at 213.36 64.77 0)
 		(fields_autoplaced yes)
 		(effects
@@
 	)
 	(label "I2C0_SDA"
-		(at 100.33 171.45 0)
+		(at 213.36 54.61 0)
 		(fields_autoplaced yes)
 		(effects
@@
 	)
 	(label "I2C0_SCL"
-		(at 100.33 173.99 0)
+		(at 213.36 57.15 0)
 		(fields_autoplaced yes)
 		(effects
@@
 	(symbol
 		(lib_id "power:GND")
-		(at 100.33 176.53 90)
+		(at 213.36 59.69 90)
 		(unit 1)
 		(exclude_from_sim no)
@@
 		(fields_autoplaced yes)
 		(property "Reference" "#PWR010"
-			(at 106.68 176.53 0)
+			(at 219.71 59.69 0)
 			(effects
 				(font
@@
 		)
 		(property "Value" "GND"
-			(at 104.14 176.5299 90)
+			(at 217.17 59.6899 90)
 			(effects
 				(font
@@
 		)
 		(property "Footprint" ""
-			(at 100.33 176.53 0)
+			(at 213.36 59.69 0)
 			(effects
 				(font
@@
 		)
 		(property "Datasheet" ""
-			(at 100.33 176.53 0)
+			(at 213.36 59.69 0)
 			(effects
 				(font
@@
 		)
 		(property "Description" "Power symbol creates a global label with name \"GND\" , ground"
-			(at 100.33 176.53 0)
+			(at 213.36 59.69 0)
 			(effects
 				(font
@@
 	(symbol
 		(lib_id "power:+3V3")
-		(at 87.63 179.07 90)
+		(at 200.66 62.23 90)
 		(unit 1)
 		(exclude_from_sim no)
@@
 		(fields_autoplaced yes)
 		(property "Reference" "#PWR013"
-			(at 91.44 179.07 0)
+			(at 204.47 62.23 0)
 			(effects
 				(font
@@
 		)
 		(property "Value" "+3V3"
-			(at 83.82 179.0699 90)
+			(at 196.85 62.2299 90)
 			(effects
 				(font
@@
 		)
 		(property "Footprint" ""
-			(at 87.63 179.07 0)
+			(at 200.66 62.23 0)
 			(effects
 				(font
@@
 		)
 		(property "Datasheet" ""
-			(at 87.63 179.07 0)
+			(at 200.66 62.23 0)
 			(effects
 				(font
@@
 		)
 		(property "Description" "Power symbol creates a global label with name \"+3V3\""
-			(at 87.63 179.07 0)
+			(at 200.66 62.23 0)
 			(effects
 				(font
@@
 			)
 		)
-		(property "Value" "1uF"
+		(property "Value" "10uF"
 			(at 64.008 27.686 0)
 			(effects
@@
 	(symbol
 		(lib_id "power:GND")
-		(at 55.88 176.53 0)
+		(at 227.33 55.88 0)
 		(unit 1)
 		(exclude_from_sim no)
@@
 		(fields_autoplaced yes)
 		(property "Reference" "#PWR012"
-			(at 55.88 182.88 0)
+			(at 227.33 62.23 0)
 			(effects
 				(font
@@
 		)
 		(property "Value" "GND"
-			(at 55.88 181.61 0)
+			(at 227.33 60.96 0)
 			(effects
 				(font
@@
 		)
 		(property "Footprint" ""
-			(at 55.88 176.53 0)
+			(at 227.33 55.88 0)
 			(effects
 				(font
@@
 		)
 		(property "Datasheet" ""
-			(at 55.88 176.53 0)
+			(at 227.33 55.88 0)
 			(effects
 				(font
@@
 		)
 		(property "Description" "Power symbol creates a global label with name \"GND\" , ground"
-			(at 55.88 176.53 0)
+			(at 227.33 55.88 0)
 			(effects
 				(font
@@
 	(symbol
 		(lib_id "Connector_Generic:Conn_01x02")
-		(at 60.96 176.53 0)
+		(at 232.41 55.88 0)
 		(mirror x)
 		(unit 1)
@@
 		(dnp no)
 		(property "Reference" "J5"
-			(at 63.5 176.5301 0)
+			(at 231.14 50.546 0)
 			(effects
 				(font
@@
 		)
 		(property "Value" "Conn_01x02"
-			(at 63.5 173.9901 0)
+			(at 226.06 50.038 0)
 			(effects
 				(font
@@
 				)
 				(justify left)
+				(hide yes)
 			)
 		)
 		(property "Footprint" "Connector_PinHeader_1.00mm:PinHeader_1x02_P1.00mm_Vertical"
-			(at 60.96 176.53 0)
+			(at 232.41 55.88 0)
 			(effects
 				(font
@@
 		)
 		(property "Datasheet" "~"
-			(at 60.96 176.53 0)
+			(at 232.41 55.88 0)
 			(effects
 				(font
@@
 		)
 		(property "Description" "Generic connector, single row, 01x02, script generated (kicad-library-utils/schlib/autogen/connector/)"
-			(at 60.96 176.53 0)
+			(at 232.41 55.88 0)
 			(effects
 				(font
@@
 		)
 		(property "Manufacturer" ""
-			(at 60.96 176.53 0)
+			(at 232.41 55.88 0)
 			(effects
 				(font
@@
 		)
 		(property "Part Number" ""
-			(at 60.96 176.53 0)
+			(at 232.41 55.88 0)
 			(effects
 				(font
@@
 	(symbol
 		(lib_id "Connector_Generic:Conn_01x01")
-		(at 30.48 177.8 180)
+		(at 261.62 55.88 180)
 		(unit 1)
 		(exclude_from_sim no)
@@
 		(fields_autoplaced yes)
 		(property "Reference" "J4"
-			(at 30.48 171.45 0)
+			(at 261.62 49.53 0)
 			(effects
 				(font
@@
 		)
 		(property "Value" "Conn_01x01"
-			(at 30.48 173.99 0)
+			(at 261.62 52.07 0)
 			(effects
 				(font
@@
 		)
 		(property "Footprint" "custom-footprints:castellated_07mm"
-			(at 30.48 177.8 0)
+			(at 261.62 55.88 0)
 			(effects
 				(font
@@
 		)
 		(property "Datasheet" "~"
-			(at 30.48 177.8 0)
+			(at 261.62 55.88 0)
 			(effects
 				(font
@@
 		)
 		(property "Description" ""
-			(at 30.48 177.8 0)
+			(at 261.62 55.88 0)
 			(effects
 				(font
@@
 		)
 		(property "Manufacturer" ""
-			(at 30.48 177.8 0)
+			(at 261.62 55.88 0)
 			(effects
 				(font
@@
 		)
 		(property "Part Number" ""
-			(at 30.48 177.8 0)
+			(at 261.62 55.88 0)
 			(effects
 				(font
@@
 	(symbol
 		(lib_id "Connector_Generic:Conn_02x06_Odd_Even")
-		(at 92.71 176.53 0)
+		(at 205.74 59.69 0)
 		(unit 1)
 		(exclude_from_sim no)
@@
 		(fields_autoplaced yes)
 		(property "Reference" "J6"
-			(at 93.98 165.1 0)
+			(at 207.01 50.8 0)
 			(effects
 				(font
@@
 		)
 		(property "Value" "Conn_02x06_Odd_Even"
-			(at 93.98 167.64 0)
+			(at 207.01 50.8 0)
 			(effects
 				(font
 					(size 1.27 1.27)
 				)
+				(hide yes)
 			)
 		)
 		(property "Footprint" "Connector_PinHeader_1.00mm:PinHeader_2x06_P1.00mm_Vertical"
-			(at 92.71 176.53 0)
+			(at 205.74 59.69 0)
 			(effects
 				(font
@@
 		)
 		(property "Datasheet" "~"
-			(at 92.71 176.53 0)
+			(at 205.74 59.69 0)
 			(effects
 				(font
@@
 		)
 		(property "Description" "Generic connector, double row, 02x06, odd/even pin numbering scheme (row 1 odd numbers, row 2 even numbers), script generated (kicad-library-utils/schlib/autogen/connector/)"
-			(at 92.71 176.53 0)
+			(at 205.74 59.69 0)
 			(effects
 				(font
@@
 		)
 		(property "Manufacturer" ""
-			(at 92.71 176.53 0)
+			(at 205.74 59.69 0)
 			(effects
 				(font
@@
 		)
 		(property "Part Number" ""
-			(at 92.71 176.53 0)
+			(at 205.74 59.69 0)
 			(effects
 				(font
@@
 			)
 		)
-		(property "Value" "10nF"
+		(property "Value" "470pF"
 			(at 58.42 30.226 0)
 			(effects
@@
 	(symbol
 		(lib_id "power:GND")
-		(at 87.63 176.53 270)
+		(at 200.66 59.69 270)
 		(unit 1)
 		(exclude_from_sim no)
@@
 		(fields_autoplaced yes)
 		(property "Reference" "#PWR09"
-			(at 81.28 176.53 0)
+			(at 194.31 59.69 0)
 			(effects
 				(font
@@
 		)
 		(property "Value" "GND"
-			(at 83.82 176.5299 90)
+			(at 196.85 59.6899 90)
 			(effects
 				(font
@@
 		)
 		(property "Footprint" ""
-			(at 87.63 176.53 0)
+			(at 200.66 59.69 0)
 			(effects
 				(font
@@
 		)
 		(property "Datasheet" ""
-			(at 87.63 176.53 0)
+			(at 200.66 59.69 0)
 			(effects
 				(font
@@
 		)
 		(property "Description" "Power symbol creates a global label with name \"GND\" , ground"
-			(at 87.63 176.53 0)
+			(at 200.66 59.69 0)
 			(effects
 				(font
